File: BoardBase.brd (EAGLE design)
At the start: 42 x 42 mm, 5 parts, among them J1 SQT-109

Commit message: Updated PQ9 to support RS-485
Connections:
- net SDA renamed D+
- removed net SCL: J1.1
- new net D-: J1.2
- net RESET: now also J1.1; no longer J1.2
Changed lines of the file:
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@@
 <signal name="IN_2">
 </signal>
-<signal name="SCL">
+<signal name="RESET">
 <contactref element="J1" pad="1"/>
 </signal>
-<signal name="SDA">
+<signal name="D+">
 <contactref element="J1" pad="3"/>
 </signal>
@@
 <wire x1="19" y1="40" x2="29" y2="40" width="0" layer="19" extent="1-1"/>
 </signal>
-<signal name="RESET">
+<signal name="D-">
 <contactref element="J1" pad="2"/>
 </signal>

Commit message: Updated template
New components from library
Parts:
- H1, H2, H3, H4: value MOUNTING-HOLE -> PQ-MOUNTING-HOLE; device Delfi-PQ:MOUNTING-HOLE -> Delfi-PQ:PQ-MOUNTING-HOLE
- J1: value SQT-109 -> CON9_SQT-109
Changed lines of the file:
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@@
 <setting verticaltext="up"/>
 </settings>
-<grid distance="0.2" unitdist="mm" unit="mm" style="lines" multiple="1" display="no" altdistance="0.02" altunitdist="mm" altunit="mm"/>
+<grid distance="0.1" unitdist="mm" unit="mm" style="lines" multiple="1" display="yes" altdistance="0.05" altunitdist="mm" altunit="mm"/>
 <layers>
 <layer number="1" name="Top" color="4" fill="1" visible="yes" active="yes"/>
@@
 <layer number="48" name="Document" color="7" fill="1" visible="yes" active="yes"/>
 <layer number="49" name="Reference" color="7" fill="1" visible="yes" active="yes"/>
+<layer number="50" name="dxf" color="7" fill="1" visible="no" active="no"/>
 <layer number="51" name="tDocu" color="7" fill="1" visible="yes" active="yes"/>
 <layer number="52" name="bDocu" color="7" fill="1" visible="yes" active="yes"/>
+<layer number="53" name="tGND_GNDA" color="7" fill="9" visible="no" active="no"/>
+<layer number="54" name="bGND_GNDA" color="1" fill="9" visible="no" active="no"/>
+<layer number="56" name="wert" color="7" fill="1" visible="no" active="no"/>
+<layer number="57" name="tCAD" color="7" fill="1" visible="no" active="no"/>
+<layer number="59" name="tCarbon" color="7" fill="1" visible="no" active="no"/>
+<layer number="60" name="bCarbon" color="7" fill="1" visible="no" active="no"/>
 <layer number="90" name="Modules" color="5" fill="1" visible="no" active="no"/>
 <layer number="91" name="Nets" color="2" fill="1" visible="no" active="no"/>
@@
 <layer number="98" name="Guide" color="6" fill="1" visible="no" active="no"/>
 <layer number="99" name="SpiceOrder" color="5" fill="1" visible="no" active="no"/>
+<layer number="100" name="Muster" color="7" fill="1" visible="no" active="no"/>
+<layer number="101" name="Patch_Top" color="12" fill="4" visible="yes" active="yes"/>
+<layer number="102" name="Vscore" color="7" fill="1" visible="yes" active="yes"/>
+<layer number="103" name="fp3" color="7" fill="1" visible="yes" active="yes"/>
+<layer number="104" name="Name" color="7" fill="1" visible="yes" active="yes"/>
+<layer number="105" name="Beschreib" color="9" fill="1" visible="yes" active="yes"/>
+<layer number="106" name="BGA-Top" color="4" fill="1" visible="yes" active="yes"/>
+<layer number="107" name="BD-Top" color="5" fill="1" visible="yes" active="yes"/>
+<layer number="108" name="fp8" color="7" fill="1" visible="yes" active="yes"/>
+<layer number="109" name="fp9" color="7" fill="1" visible="yes" active="yes"/>
+<layer number="110" name="fp0" color="7" fill="1" visible="yes" active="yes"/>
+<layer number="111" name="LPC17xx" color="7" fill="1" visible="yes" active="yes"/>
+<layer number="112" name="tSilk" color="7" fill="1" visible="yes" active="yes"/>
+<layer number="113" name="ReferenceLS" color="7" fill="1" visible="no" active="no"/>
+<layer number="116" name="Patch_BOT" color="9" fill="4" visible="yes" active="yes"/>
+<layer number="118" name="Rect_Pads" color="7" fill="1" visible="no" active="no"/>
+<layer number="121" name="_tsilk" color="7" fill="1" visible="yes" active="yes"/>
+<layer number="122" name="_bsilk" color="7" fill="1" visible="yes" active="yes"/>
+<layer number="123" name="tTestmark" color="7" fill="1" visible="yes" active="yes"/>
+<layer number="124" name="bTestmark" color="7" fill="1" visible="yes" active="yes"/>
+<layer number="125" name="_tNames" color="7" fill="1" visible="yes" active="yes"/>
+<layer number="126" name="_bNames" color="7" fill="1" visible="yes" active="yes"/>
+<layer number="127" name="_tValues" color="7" fill="1" visible="yes" active="yes"/>
+<layer number="128" name="_bValues" color="7" fill="1" visible="yes" active="yes"/>
+<layer number="129" name="Mask" color="7" fill="1" visible="yes" active="yes"/>
+<layer number="130" name="130bmp" color="7" fill="1" visible="yes" active="yes"/>
+<layer number="131" name="tAdjust" color="7" fill="1" visible="yes" active="yes"/>
+<layer number="132" name="bAdjust" color="7" fill="1" visible="yes" active="yes"/>
+<layer number="144" name="Drill_legend" color="7" fill="1" visible="yes" active="yes"/>
+<layer number="145" name="DrillLegend_01-16" color="7" fill="1" visible="yes" active="yes"/>
+<layer number="150" name="Notes" color="7" fill="1" visible="yes" active="yes"/>
+<layer number="151" name="HeatSink" color="7" fill="1" visible="yes" active="yes"/>
+<layer number="152" name="_bDocu" color="7" fill="1" visible="yes" active="yes"/>
+<layer number="153" name="FabDoc1" color="6" fill="1" visible="no" active="no"/>
+<layer number="154" name="FabDoc2" color="2" fill="1" visible="no" active="no"/>
+<layer number="155" name="FabDoc3" color="7" fill="15" visible="no" active="no"/>
+<layer number="199" name="Contour" color="7" fill="1" visible="yes" active="yes"/>
+<layer number="200" name="200bmp" color="1" fill="10" visible="yes" active="yes"/>
+<layer number="201" name="201bmp" color="2" fill="1" visible="no" active="no"/>
+<layer number="202" name="202bmp" color="3" fill="1" visible="no" active="no"/>
+<layer number="203" name="203bmp" color="4" fill="10" visible="yes" active="yes"/>
+<layer number="204" name="204bmp" color="5" fill="10" visible="yes" active="yes"/>
+<layer number="205" name="205bmp" color="6" fill="10" visible="yes" active="yes"/>
+<layer number="206" name="206bmp" color="7" fill="10" visible="yes" active="yes"/>
+<layer number="207" name="207bmp" color="8" fill="10" visible="yes" active="yes"/>
+<layer number="208" name="208bmp" color="9" fill="10" visible="yes" active="yes"/>
+<layer number="209" name="209bmp" color="7" fill="1" visible="yes" active="yes"/>
+<layer number="210" name="210bmp" color="7" fill="1" visible="yes" active="yes"/>
+<layer number="211" name="211bmp" color="7" fill="1" visible="yes" active="yes"/>
+<layer number="212" name="212bmp" color="7" fill="1" visible="yes" active="yes"/>
+<layer number="213" name="213bmp" color="7" fill="1" visible="yes" active="yes"/>
+<layer number="214" name="214bmp" color="7" fill="1" visible="yes" active="yes"/>
+<layer number="215" name="215bmp" color="7" fill="1" visible="yes" active="yes"/>
+<layer number="216" name="216bmp" color="7" fill="1" visible="yes" active="yes"/>
+<layer number="217" name="217bmp" color="18" fill="1" visible="no" active="no"/>
+<layer number="218" name="218bmp" color="19" fill="1" visible="no" active="no"/>
+<layer number="219" name="219bmp" color="20" fill="1" visible="no" active="no"/>
+<layer number="220" name="220bmp" color="21" fill="1" visible="no" active="no"/>
+<layer number="221" name="221bmp" color="22" fill="1" visible="no" active="no"/>
+<layer number="222" name="222bmp" color="23" fill="1" visible="no" active="no"/>
+<layer number="223" name="223bmp" color="24" fill="1" visible="no" active="no"/>
+<layer number="224" name="224bmp" color="25" fill="1" visible="no" active="no"/>
+<layer number="225" name="225bmp" color="7" fill="1" visible="yes" active="yes"/>
+<layer number="226" name="226bmp" color="7" fill="1" visible="yes" active="yes"/>
+<layer number="227" name="227bmp" color="7" fill="1" visible="yes" active="yes"/>
+<layer number="228" name="228bmp" color="7" fill="1" visible="yes" active="yes"/>
+<layer number="229" name="229bmp" color="7" fill="1" visible="yes" active="yes"/>
+<layer number="230" name="230bmp" color="7" fill="1" visible="yes" active="yes"/>
+<layer number="231" name="Eagle3D_PG1" color="7" fill="1" visible="no" active="no"/>
+<layer number="232" name="Eagle3D_PG2" color="7" fill="1" visible="no" active="no"/>
+<layer number="233" name="Eagle3D_PG3" color="7" fill="1" visible="no" active="no"/>
+<layer number="248" name="Housing" color="7" fill="1" visible="yes" active="yes"/>
+<layer number="249" name="Edge" color="7" fill="1" visible="yes" active="yes"/>
+<layer number="250" name="Descript" color="7" fill="1" visible="no" active="no"/>
+<layer number="251" name="SMDround" color="7" fill="1" visible="no" active="no"/>
+<layer number="254" name="cooling" color="7" fill="1" visible="yes" active="yes"/>
+<layer number="255" name="routoute" color="7" fill="1" visible="yes" active="yes"/>
 </layers>
 <board>
@@
 </autorouter>
 <elements>
-<element name="J1" library="Delfi-PQ" package="SQT-109" value="SQT-109" x="21" y="40" locked="yes"/>
-<element name="H1" library="Delfi-PQ" package="MOUNTING-HOLE" value="MOUNTING-HOLE" x="3" y="39" locked="yes">
+<element name="J1" library="Delfi-PQ" package="SQT-109" value="CON9_SQT-109" x="21" y="40" locked="yes"/>
+<element name="H1" library="Delfi-PQ" package="PQ-MOUNTING-HOLE" value="PQ-MOUNTING-HOLE" x="3" y="39" locked="yes">
 <attribute name="HEIGHT" value="-1" x="3" y="39" size="1.778" layer="27" display="off"/>
 </element>
-<element name="H2" library="Delfi-PQ" package="MOUNTING-HOLE" value="MOUNTING-HOLE" x="39" y="39" locked="yes">
+<element name="H2" library="Delfi-PQ" package="PQ-MOUNTING-HOLE" value="PQ-MOUNTING-HOLE" x="39" y="39" locked="yes">
 <attribute name="HEIGHT" value="-1" x="39" y="39" size="1.778" layer="27" display="off"/>
 </element>
-<element name="H3" library="Delfi-PQ" package="MOUNTING-HOLE" value="MOUNTING-HOLE" x="39" y="3" locked="yes">
+<element name="H3" library="Delfi-PQ" package="PQ-MOUNTING-HOLE" value="PQ-MOUNTING-HOLE" x="39" y="3" locked="yes">
 <attribute name="HEIGHT" value="-1" x="39" y="3" size="1.778" layer="27" display="off"/>
 </element>
-<element name="H4" library="Delfi-PQ" package="MOUNTING-HOLE" value="MOUNTING-HOLE" x="3" y="3" locked="yes">
+<element name="H4" library="Delfi-PQ" package="PQ-MOUNTING-HOLE" value="PQ-MOUNTING-HOLE" x="3" y="3" locked="yes">
 <attribute name="HEIGHT" value="-1" x="3" y="3" size="1.778" layer="27" display="off"/>
 </element>

Commit message: Renamed mounting holes
Parts:
- H1, H2, H3, H4: value PQ-MOUNTING-HOLE -> MOUNTING-HOLE_PQ; device Delfi-PQ:PQ-MOUNTING-HOLE -> Delfi-PQ:MOUNTING-HOLE-PQ
Changed lines of the file:
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@@
 <layer number="112" name="tSilk" color="7" fill="1" visible="yes" active="yes"/>
 <layer number="113" name="ReferenceLS" color="7" fill="1" visible="no" active="no"/>
+<layer number="114" name="Al_Dimension" color="7" fill="1" visible="yes" active="yes"/>
+<layer number="115" name="Countersink" color="7" fill="1" visible="yes" active="yes"/>
 <layer number="116" name="Patch_BOT" color="9" fill="4" visible="yes" active="yes"/>
 <layer number="118" name="Rect_Pads" color="7" fill="1" visible="no" active="no"/>
@@
 </autorouter>
 <elements>
-<element name="J1" library="Delfi-PQ" package="SQT-109" value="CON9_SQT-109" x="21" y="40" locked="yes"/>
-<element name="H1" library="Delfi-PQ" package="PQ-MOUNTING-HOLE" value="PQ-MOUNTING-HOLE" x="3" y="39" locked="yes">
-<attribute name="HEIGHT" value="-1" x="3" y="39" size="1.778" layer="27" display="off"/>
-</element>
-<element name="H2" library="Delfi-PQ" package="PQ-MOUNTING-HOLE" value="PQ-MOUNTING-HOLE" x="39" y="39" locked="yes">
-<attribute name="HEIGHT" value="-1" x="39" y="39" size="1.778" layer="27" display="off"/>
-</element>
-<element name="H3" library="Delfi-PQ" package="PQ-MOUNTING-HOLE" value="PQ-MOUNTING-HOLE" x="39" y="3" locked="yes">
-<attribute name="HEIGHT" value="-1" x="39" y="3" size="1.778" layer="27" display="off"/>
-</element>
-<element name="H4" library="Delfi-PQ" package="PQ-MOUNTING-HOLE" value="PQ-MOUNTING-HOLE" x="3" y="3" locked="yes">
-<attribute name="HEIGHT" value="-1" x="3" y="3" size="1.778" layer="27" display="off"/>
+<element name="J1" library="Delfi-PQ" package="SQT-109" value="CON9_SQT-109" x="21" y="40" locked="yes">
+<attribute name="HEIGHT" value="7.0" x="21" y="40" size="1.778" layer="27" display="off"/>
+</element>
+<element name="H1" library="Delfi-PQ" package="MOUNTING-HOLE-PQ" value="MOUNTING-HOLE_PQ" x="3" y="39" locked="yes">
+<attribute name="HEIGHT" value="7.0" x="3" y="39" size="1.778" layer="27" display="off"/>
+</element>
+<element name="H2" library="Delfi-PQ" package="MOUNTING-HOLE-PQ" value="MOUNTING-HOLE_PQ" x="39" y="39" locked="yes">
+<attribute name="HEIGHT" value="7.0" x="39" y="39" size="1.778" layer="27" display="off"/>
+</element>
+<element name="H3" library="Delfi-PQ" package="MOUNTING-HOLE-PQ" value="MOUNTING-HOLE_PQ" x="39" y="3" locked="yes">
+<attribute name="HEIGHT" value="7.0" x="39" y="3" size="1.778" layer="27" display="off"/>
+</element>
+<element name="H4" library="Delfi-PQ" package="MOUNTING-HOLE-PQ" value="MOUNTING-HOLE_PQ" x="3" y="3" locked="yes">
+<attribute name="HEIGHT" value="7.0" x="3" y="3" size="1.778" layer="27" display="off"/>
 </element>
 </elements>
